File: eagle/ctia.sch (EAGLE design)
At the start: 6 parts, among them IC1 IVC102U, X1 BU-SMA-V

Commit message: board/solid works
Parts:
- removed DATA: (no value), con-molex:KK-156-5
- removed POWER: (no value), con-molex:KK-156-3
- removed X1: BU-SMA-V, con-coax:BU-SMA-V
- added R1: (no value), resistor:R-US_0207/12
- added R2: (no value), resistor:R-US_0207/10
- added X5: (no value), con-subd:F09HP
- IC1: value IVC102U -> IVC102UADAPTOR; device burr-brown:IVC102U -> burr-brown:IVC102UADAPTOR
- U$1: value ADS1015 -> CTIA; device texas:ADS1015 -> ctia:CTIA
Connections:
- removed net -5V: IC1.V-, POWER-1.S
- removed net N$5: IC1.IN, X1.1
- removed net N$6: IC1.VOUT, U$1.AIN0
- removed net N$7: DATA-1.S, U$1.SCL
- removed net N$8: DATA-2.S, U$1.SDA
- new net +15V: IC1.V+, X5.1
- new net -15V: IC1.V-, X5.4
- new net VIN: IC1.IN, U$1.P$1
- new net VOUT: IC1.VOUT, X5.8
- net +5V: now also R1.1, R2.1, X5.5; no longer IC1.V+, POWER-3.S, U$1.ADDR, U$1.VDD
- net GND: now also X5.2, X5.3, X5.9; no longer DATA-3.S, POWER-2.S, U$1.AIN1, U$1.GND, X1.2
- net RESET: now also R2.2, X5.6; no longer DATA-5.S
- net SAMPLE: now also R1.2, X5.7; no longer DATA-4.S
Other:
- note removed: "i2c address 0x49"
