File: eagle/untitled.brd (EAGLE design)
At the start: 69.8 x 65.7 mm, 9 parts, among them IC1 IVC102UADAPTOR

Commit message: board/solid works
Parts:
- added C1, C2, C6, C7: .1u, resistor:C050-050X075
- added C10, C5: .68n, resistor:C075-032X103
- added C3, C8: gimmick, resistor:C075-032X103
- added C4, C9: 150p, resistor:C075-032X103
- added IC2, IC3: LF442N, linear:DIL08
- added IC4: IVC102UADAPTOR, burr-brown:DIL14
- added R10, R3, R5, R8: 1M, resistor:0207/10
- added R11, R6: 649, resistor:0207/10
- added R12, R7: 50k, pot:RJ9W
- added R13: (no value), resistor:0207/12
- added R14: (no value), resistor:0207/10
- added R4, R9: 10M, resistor:0207/10
- added SW1: (no value), special:EDG-03
- added X10, X11, X13, X14, X15, X16, X7, X8: (no value), con-molex:KK-156-2
- added X12, X5, X9: (no value), con-molex:KK-156-6
Connections:
- new net +15V1: C1.1, IC2.8, R7.E, X5.6
- new net +15V2: C6.1, IC3.8, R12.E, X9.6
- new net +15V3: IC4.14, X12.6
- new net +5V1: X5.4, X5.5
- new net +5V2: X9.4, X9.5
- new net +5V3: R13.1, R14.1, X12.4, X12.5
- new net -15V1: C2.1, IC2.4, R7.A, X5.1
- new net -15V2: C7.1, IC3.4, R12.A, X9.1
- new net -15V3: IC4.9, X12.1
- new net GND1: C1.2, C2.2, R6.2, X5.2, X5.3, X7.2, X8.2
- new net GND2: C6.2, C7.2, R11.2, X10.2, X11.2, X9.2, X9.3
- new net GND3: IC4.1, IC4.13, X12.2, X12.3, X13.1, X14.1, X15.2, X16.2
- new net N$10: C4.2, IC2.3, R5.2, R6.1
- new net N$11: R5.1, R7.S
- new net N$12: C10.1, C8.2, IC3.2, R8.2, R9.1
- new net N$13: C8.1, C9.1, IC3.1, R9.2, X10.1
- new net N$14: C10.2, R8.1, X11.1
- new net N$15: C9.2, IC3.3, R10.2, R11.1
- new net N$16: R10.1, R12.S
- new net N$17: IC4.6, SW1.1
- new net N$18: IC4.5, SW1.2
- new net N$19: IC4.4, SW1.3
- new net N$20: IC4.3, SW1.4, SW1.5, SW1.6
- new net N$21: IC4.2, X15.1
- new net N$22: IC4.10, X16.1
- new net N$7: C3.2, C5.1, IC2.2, R3.2, R4.1
- new net N$8: C3.1, C4.1, IC2.1, R4.2, X7.1
- new net N$9: C5.2, R3.1, X8.1
- new net RESET1: IC4.12, R14.2, X13.2
- new net SAMPLE1: IC4.11, R13.2, X14.2
Routing:
- net -15V2: track 0.00 -> 52.8 mm
- net -15V1: track 0.00 -> 52.8 mm
- net -15V3: track 0.00 -> 48.2 mm
- net +5V3: track 0.00 -> 44.0 mm
- net N$12: track 0.00 -> 41.5 mm
- net N$7: track 0.00 -> 41.5 mm
- net +15V2: track 0.00 -> 41.5 mm
- net +15V1: track 0.00 -> 41.5 mm
- net N$13: track 0.00 -> 40.2 mm
- net N$8: track 0.00 -> 40.2 mm
- net N$21: track 0.00 -> 38.5 mm
- net RESET1: track 0.00 -> 38.2 mm
- net SAMPLE1: track 0.00 -> 33.3 mm
- net N$22: track 0.00 -> 28.7 mm
- net N$20: track 0.00 -> 27.2 mm
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- added copper zone on layer 16, net GND1
- added copper zone on layer 16, net GND2
- added copper zone on layer 16, net GND3
Other:
- board size 69.8 x 65.7 mm -> 132.1 x 143.5 mm
